File: hardware/LoRaNode_STM32G474RE/LoRaNode_STM32G474RE.kicad_sch (KiCad schematic)
At the start: 4 parts

Commit message: feat: complete hardware v1 (ERC almost clean) and initial firmware peripherals config
Other:
- sheet SSD1306{I2C} renamed I2C1{SCL SDA}
- sheet I2C1{SCL SDA} ports: added I2C1{SCL SDA}; removed SSD1306{I2C}
- sheet STM32 ports: added I2C1{SCL SDA}; removed SSD1306{I2C}
Changed lines of the file:
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@@
 	(bus
 		(pts
-			(xy 113.03 58.42) (xy 133.35 58.42)
+			(xy 113.03 57.15) (xy 133.35 57.15)
 		)
 		(stroke
@@
 	(bus
 		(pts
-			(xy 113.03 58.42) (xy 113.03 52.07)
-		)
-		(stroke
-			(width 0)
-			(type default)
-		)
-	)
-	(wire
-		(pts
-			(xy 95.25 101.6) (xy 102.87 101.6)
+			(xy 113.03 57.15) (xy 113.03 52.07)
+		)
+		(stroke
+			(width 0)
+			(type default)
+		)
+	)
+	(wire
+		(pts
+			(xy 69.85 101.6) (xy 102.87 101.6)
 		)
 		(stroke
@@
 	(wire
 		(pts
-			(xy 95.25 114.3) (xy 130.81 114.3)
+			(xy 69.85 114.3) (xy 130.81 114.3)
 		)
 		(stroke
@@
 	)
 	(sheet
-		(at 76.2 97.79)
+		(at 50.8 97.79)
 		(size 19.05 6.35)
 		(exclude_from_sim no)
@@
 		)
 		(property "Sheetname" "BTN_BOOT"
-			(at 76.2 97.0784 0)
+			(at 50.8 97.0784 0)
 			(effects
 				(font
@@
 		)
 		(property "Sheetfile" "BTN_BOOT.kicad_sch"
-			(at 76.2 104.7246 0)
+			(at 50.8 104.7246 0)
 			(effects
 				(font
@@
 		)
 		(pin "BTN_BOOT" input
-			(at 95.25 101.6 0)
+			(at 69.85 101.6 0)
 			(effects
 				(font
@@
 			(color 0 0 0 0.0000)
 		)
-		(property "Sheetname" "SSD1306{I2C}"
+		(property "Sheetname" "I2C1{SCL SDA}"
 			(at 196.85 53.8984 0)
 			(effects
@@
 			)
 		)
-		(pin "SSD1306{I2C}" bidirectional
+		(pin "I2C1{SCL SDA}" bidirectional
 			(at 196.85 59.69 180)
 			(effects
@@
 	)
 	(sheet
-		(at 76.2 110.49)
+		(at 50.8 110.49)
 		(size 19.05 6.35)
 		(exclude_from_sim no)
@@
 		)
 		(property "Sheetname" "BTN_RST"
-			(at 76.2 109.7784 0)
+			(at 50.8 109.7784 0)
 			(effects
 				(font
@@
 		)
 		(property "Sheetfile" "BTN_RST.kicad_sch"
-			(at 76.2 117.4246 0)
+			(at 50.8 117.4246 0)
 			(effects
 				(font
@@
 		)
 		(pin "NRST" input
-			(at 95.25 114.3 0)
+			(at 69.85 114.3 0)
 			(effects
 				(font
@@
 			)
 		)
-		(pin "SSD1306{I2C}" bidirectional
+		(pin "I2C1{SCL SDA}" bidirectional
 			(at 176.53 62.23 0)
 			(effects
@@
 		)
 		(pin "RFM95{MISO MOSI SCK NSS RST DIO0}" bidirectional
-			(at 133.35 58.42 180)
-			(effects
-				(font
+			(at 133.35 57.15 180)
+			(effects
+				(font
