File: hardware/LoRaNode_STM32G474RE/STM32.kicad_sch (KiCad schematic)
At the start: 15 parts, among them U4 STM32G474RETx, Y2 24mHz 8pf

Commit message: feat: complete hardware v1 (ERC almost clean) and initial firmware peripherals config
Connections:
- net SSD1306.SCL is gone; now on net I2C1.SCL: R22.2
- net SSD1306.SDA is gone; now on net I2C1.SDA: R20.2
- net I2C1.SDA: now reaches U4.51 (PA15)
- net I2C1.SCL: now reaches U4.60 (PB7)
- no-connect marks 41 -> 37
Other:
- moved on the sheet: C17, C18, C19, C20, C21, C22, C23, C24, C25, R19, R20, R21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
